File: esp-doorbell.kicad_sch (KiCad schematic)
At the start: 42 parts, among them J1 Screw_Terminal_01x02, J2 Conn_01x07_Socket, J3 Conn_01x07_Socket, J4 Screw_Terminal_01x02, J5 Screw_Terminal_01x02, K2 JQC-3FF-005-1Z, Q1 NMOS, U2 TPS5430DDA

Commit message: fix schematics, add layout
Parts:
- removed FID1, FID2, FID3: Fiducial, Fiducial:Fiducial_0.5mm_Mask1.5mm, symbol Mechanical:Fiducial
- removed H4: MountingHole_Pad, MountingHole:MountingHole_3.2mm_M3_DIN965_Pad, symbol Mechanical:MountingHole_Pad
- removed J2, J3: Conn_01x07_Socket, Connector_PinSocket_2.54mm:PinSocket_1x07_P2.54mm_Vertical, symbol Connector_Generic:Conn_01x07
- removed U1: ~, Library:XIAO-ESP32C6-DIP, symbol New_Library:Seed_Studio_Xiao_ESP32C6
- added U2: XIAO-ESP32-S3-SMD, Seeed Studio XIAO Series Library:XIAO-ESP32C6-SMD, symbol Seeed_Studio_XIAO_Series:XIAO-ESP32-C6-SMD
- F1: footprint (none) -> LED_SMD:LED_1206_3216Metric
- renumbered C4 to C1, C5 to C2, C6 to C3, C8 to C4, C7 to C5, C3 to C6, C2 to C7, D5 to D1, D4 to D3, D1 to D4, D6 to D5, D3 to D6, J4 to J2, J5 to J3, K2 to K1, R3 to R1, R1 to R2, R8 to R3, R7 to R4, R2 to R5, R5 to R6, R11 to R7, R9 to R8, R6 to R9, TP2 to TP1, TP1 to TP2, U2 to U1
Connections:
- net +3V3: now also U2.12 (3V3)
- net +5V: now also U2.14 (5V)
- net AC1: now also J3.2 (Pin_2); no longer J3.1 (Pin_1), K1.11
- net AC2: no longer J3.2 (Pin_2)
- net D0: now also U2.1 (GPIO0_A0_D0)
- net D1: now also U2.2 (GPIO1_A1_D1)
- net D2: now also U2.3 (GPIO2_A2_D2)
- net GND: now also U2.13 (GND), U2.16 (GND)
- new net: J3.1 (Pin_1), K1.11
- no-connect marks 10 -> 19
Other:
- note added: "User LED"
- note removed: "user led"
- moved on the sheet: C7, D5, D6, H1, H2, H3, R8, R9

Commit message: make board a bit smaller
Connections:
- net GND: no longer U2.16 (GND)
- no-connect marks 19 -> 20
Changed lines of the file:
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@@
+	)
+	(no_connect
+		(at 219.71 74.93)
 	)
 	(no_connect
@@
 		)
 		(stroke
-			(width 0)
-			(type default)
-		)
-	)
-	(wire
-		(pts
-			(xy 219.71 74.93) (xy 219.71 83.82)
-		)
-		(stroke
